Commit message: feat: migration from Gazebo classic to Gazebo

File: twr_description/urdf/ros2_control.xacro (robot description, xacro)
@@ -1,9 +1,9 @@
 <?xml version="1.0"?>
 <robot xmlns:xacro="http://www.ros.org/wiki/xacro" >
-    <ros2_control>
+    <ros2_control name="twr diff" type="system">
         <hardware>
-            <!-- name of hardware interface
-            it will talk to Gazebo just like a normal hardware interface -->
-            <plugin> gazebo_ros2_control/GazeboSystem </plugin>
+            <!-- name of hardware interface -->
+            <!-- it will talk to Gazebo just like a normal hardware interface -->
+            <plugin> gz_ros2_control/GazeboSystem </plugin>
         </hardware>
         <joint name="left_wheel_joint">
@@ -25,5 +25,5 @@
     </ros2_control>
     <gazebo>
-        <plugin name="gazebo_ros2_control" filename="libgazebo_ros2_control.so">
+        <plugin filename="libgz_ros2_control-system.so" name="gz_ros2_control::GazeboSimROS2ControlPlugin">
             <parameters> $(find twr_description)/controllers/twr_diff_drive.yaml </parameters>
         </plugin>

File: twr_description/urdf/twr.urdf.xacro (robot description, xacro)
@@ -1,7 +1,8 @@
 <?xml version="1.0"?>
 <robot name="twr" xmlns:xacro="http://ros.org/wiki/xacro">
+    <!-- Include files -->
     <xacro:include filename="_inertia.macro.xacro"/>
     <xacro:include filename="_colors.xacro"/>
-    <xacro:include filename="ros2_control.xacro"/>
+    <!-- <xacro:include filename="ros2_control.xacro"/> -->
     <xacro:property name="mm2m" value="0.001"/>
     <xacro:property name="base_length" value="${200*mm2m}"/>
@@ -41,11 +42,4 @@
         </xacro:box_inertia>
     </link>
-    <!-- === CHASSIS === -->
-    <!-- <joint name="chassis_joint" type="fixed">
-        <parent link="base_link"/>
-        <child link="chassis_link" />
-        <origin xyz="0 0 0" rpy="0 0 0"/>
-    </joint>
-    <link name="chassis_link"></link> -->
     <!-- ============== -->
     <!-- === WHEELS === -->
@@ -150,3 +144,7 @@
         </xacro:sphere_inertia>
     </link>
+    <!-- Joint states plugin -->
+    <gazebo>
+        <plugin filename="gz-sim-joint-state-publisher-system" name="gz::sim::systems::JointStatePublisher"/>
+    </gazebo>
 </robot>
