Commit message: refactor(urdf): generalization of macro for inertia.macro.xacro file

File: twr_description/urdf/_inertia.macro.xacro (robot description, xacro)
@@ -1,32 +1,29 @@
 <?xml version="1.0"?>
 <robot xmlns:xacro="http://www.ros.org/wiki/xacro" >
-    <xacro:macro name="box_inertia" params="m l w h *origin">
+    <xacro:macro name="inertia" params="shape xyz rpy l:=0 w:=0 h:=0 r:=0 m:=0">
         <inertial>
             <mass value="${m}"/>
-            <inertia
-                ixx="${(m/12) * (h*h + l*l)}" ixy="0.0" ixz="0.0"
-                iyy="${(m/12) * (w*w + l*l)}" iyz="0.0"
-                izz="${(m/12) * (w*w + h*h)}" />
-        </inertial>
-        <xacro:insert_block name="origin"/>
-    </xacro:macro>
-    <xacro:macro name="cylinder_inertia" params="m r l *origin">
-        <inertial>
-            <mass value="${m}"/>
-            <inertia
-                ixx="${m*l*l/12 + m*r*r/4}" ixy="0.0" ixz="0.0"
-                iyy="${m*l*l/12 + m*r*r/4}" iyz="0.0"
-                izz="${m*r*r/2}" />
-            <xacro:insert_block name="origin"/>
-        </inertial>
-    </xacro:macro>
-    <xacro:macro name="sphere_inertia" params="m r *origin">
-        <inertial>
-            <mass value="${m}"/>
-            <inertia
-                ixx="${m*r*r*2/5}" ixy="0.0" ixz="0.0"
-                iyy="${m*r*r*2/5}" iyz="0.0"
-                izz="${m*r*r*2/5}" />
-                <xacro:insert_block name="origin"/>
+            <xacro:if value="${shape == 'box'}">
+                <inertia
+                    ixx="${m/12 * (h*h + l*l)}" ixy="0.0" ixz="0.0"
+                    iyy="${m/12 * (w*w + l*l)}" iyz="0.0"
+                    izz="${m/12 * (w*w + h*h)}"
+                />
+            </xacro:if>
+            <xacro:if value="${shape == 'cylinder'}">
+                <inertia
+                    ixx="${m*w*w/12 + m*r*r/4}" ixy="0.0" ixz="0.0"
+                    iyy="${m*w*w/12 + m*r*r/4}" iyz="0.0"
+                    izz="${m*r*r/2}"
+                />
+            </xacro:if>
+            <xacro:if value="${shape == 'sphere'}">
+                <inertia
+                    ixx="${m*r*r*2/5}" ixy="0.0" ixz="0.0"
+                    iyy="${m*r*r*2/5}" iyz="0.0"
+                    izz="${m*r*r*2/5}"
+                />
+            </xacro:if>
+            <origin xyz="${xyz}" rpy="${rpy}"/>
         </inertial>
     </xacro:macro>

File: twr_description/urdf/twr.urdf.xacro (robot description, xacro)
@@ -6,5 +6,5 @@
     <xacro:include filename="ros2_control.xacro"/>
     <xacro:include filename="gz.xacro"/>
-    <xacro:include filename="wheel.xacro"/>
+    <xacro:include filename="wheel.macro.xacro"/>
     <xacro:property name="mm2m" value="0.001"/>
     <xacro:property name="base_length" value="${200*mm2m}"/>
@@ -40,7 +40,5 @@
             <origin xyz="0 0 0" rpy="0 0 0"/>
         </collision>
-        <xacro:box_inertia m="1" l="${base_length}" w="${base_width}"  h="${base_height}">
-            <origin xyz="0 0 0" rpy="0 0 0"/>
-        </xacro:box_inertia>
+        <xacro:inertia shape="box" xyz="0 0 0" rpy="0 0 0" l="${base_length}" w="${base_width}" h="${base_height}" m="1"/>
     </link>
     <!-- ============== -->

File: twr_description/urdf/wheel.macro.xacro (robot description, xacro)
@@ -26,7 +26,5 @@
                     <origin xyz="0 0 0" rpy="0 0 0"/>
                 </collision>
-                <xacro:cylinder_inertia m="${m}" r="${radius}" l="${width}">
-                    <origin xyz="0 0 0" rpy="0 0 0"/>
-                </xacro:cylinder_inertia>
+                <xacro:inertia shape="cylinder" xyz="0 0 0" rpy="0 0 0" r="${radius}" w="${width}" m="${m}"/>
             </link>
         </xacro:if>
@@ -54,7 +52,5 @@
                     <origin xyz="0 0 0" rpy="0 0 0"/>
                 </collision>
-                <xacro:sphere_inertia m="${m}" r="${radius}">
-                    <origin xyz="0 0 0" rpy="0 0 0"/>
-                </xacro:sphere_inertia>
+                <xacro:inertia shape="sphere" xyz="0 0 0" rpy="0 0 0" r="${radius}" m="${m}"/>
             </link>
         </xacro:if>
