Commit message: fix: update urdf description, incorrect axes orientation for wheels

File: twr_description/urdf/gz.xacro (robot description, xacro)
@@ -2,12 +2,12 @@
 <robot xmlns:xacro="http://www.ros.org/wiki/xacro">
     <!-- Joint states plugin -->
-    <gazebo>
+    <!-- <gazebo>
         <plugin filename="gz-sim-joint-state-publisher-system" name="gz::sim::systems::JointStatePublisher"/>
-    </gazebo>
+    </gazebo> -->
     <!-- Ros2 control plugin -->
     <!-- In addition to the ros2_control tags, a Gazebo plugin needs to be added to your URDF
     that actually parses the ros2_control tags and loads the appropriate hardware interfaces and controller manager -->
     <gazebo>
-        <plugin filename="libgz_ros2_control-system.so" name="gz_ros2_control::GazeboSimROS2ControlPlugin">
+        <plugin filename="gz_ros2_control-system" name="gz_ros2_control::GazeboSimROS2ControlPlugin">
             <parameters> $(find twr_description)/controllers/twr_diff_drive.yaml </parameters>
         </plugin>

File: twr_description/urdf/twr.urdf.xacro (robot description, xacro)
@@ -16,10 +16,10 @@
     <!-- === WORLD === -->
     <!-- ============= -->
-    <link name="world_link"/>
+    <link name="odom"/>
     <!-- ============ -->
     <!-- === BASE === -->
     <!-- ============ -->
     <joint name="base_joint" type="fixed">
-        <parent link="world_link"/>
+        <parent link="odom"/>
         <child link="base_link" />
         <origin xyz="0 0 ${wheel_radius+0.01}" rpy="0 0 0"/>
@@ -73,5 +73,5 @@
         <parent link="base_link"/>
         <child link="right_wheel_link" />
-        <origin xyz="0 -${base_width/2 + wheel_width/2 + 0.01} 0" rpy="${pi/2} 0 0"/>
+        <origin xyz="0 -${base_width/2 + wheel_width/2 + 0.01} 0" rpy="-${pi/2} 0 0"/>
         <axis xyz="0 0 1"/>
     </joint>
@@ -97,5 +97,5 @@
     <!-- === CASTER WHEELS === -->
     <!-- ===================== -->
-    <joint name="caster_front_wheel_joint" type="continuous">
+    <joint name="caster_front_wheel_joint" type="fixed">
         <parent link="base_link"/>
         <child link="caster_front_wheel_link"/>
@@ -121,5 +121,5 @@
         </xacro:sphere_inertia>
     </link>
-    <joint name="caster_back_wheel_joint" type="continuous">
+    <joint name="caster_back_wheel_joint" type="fixed">
         <parent link="base_link"/>
         <child link="caster_back_wheel_link"/>

Commit message: feat: add 2D LIDAR urdf

File: twr_description/urdf/gz.xacro (robot description, xacro)
@@ -1,15 +1,41 @@
 <?xml version="1.0"?>
 <robot xmlns:xacro="http://www.ros.org/wiki/xacro">
-    <!-- Joint states plugin -->
-    <!-- <gazebo>
-        <plugin filename="gz-sim-joint-state-publisher-system" name="gz::sim::systems::JointStatePublisher"/>
-    </gazebo> -->
-    <!-- Ros2 control plugin -->
-    <!-- In addition to the ros2_control tags, a Gazebo plugin needs to be added to your URDF
-    that actually parses the ros2_control tags and loads the appropriate hardware interfaces and controller manager -->
+    <!-- === Plugins === -->
     <gazebo>
+        <!-- Ros2 control plugin -->
+        <!-- In addition to the ros2_control tags, a Gazebo plugin needs to be added to your URDF
+        that actually parses the ros2_control tags and loads the appropriate hardware interfaces and controller manager -->
         <plugin filename="gz_ros2_control-system" name="gz_ros2_control::GazeboSimROS2ControlPlugin">
             <parameters> $(find twr_description)/controllers/twr_diff_drive.yaml </parameters>
         </plugin>
+        <plugin filename="gz-sim-sensors-system" name="gz::sim::systems::Sensors">
+            <render_engine>ogre2</render_engine>
+        </plugin>
+    </gazebo>
+    <!-- =============== -->
+    <!-- === SENSORS === -->
+    <!-- =============== -->
+    <!-- === LIDAR === -->
+    <gazebo reference="lidar_link">
+        <sensor name="lidar_link" type="gpu_lidar">
+            <pose> 0 0 0 0 0 0 </pose>
+            <visualize>true</visualize>
+            <update_rate>10</update_rate>
+            <lidar>
+                <scan>
+                    <horizontal>
+                        <samples>360</samples>
+                        <min_angle>-3.1415926535</min_angle>
+                        <max_angle>3.1415926535</max_angle>
+                    </horizontal>
+                </scan>
+                <range>
+                    <min>0.3</min>
+                    <max>10</max>
+                </range>
+            </lidar>
+            <topic>scan</topic>
+            <!-- <gz_frame_id>lidar_link</gz_frame_id> -->
+        </sensor>
     </gazebo>
 </robot>

File: twr_description/urdf/twr.urdf.xacro (robot description, xacro)
@@ -7,4 +7,5 @@
     <xacro:include filename="gz.xacro"/>
     <xacro:include filename="wheel.macro.xacro"/>
+    <xacro:include filename="twr_lidar.xacro"/>
     <xacro:property name="mm2m" value="0.001"/>
     <xacro:property name="base_length" value="${200*mm2m}"/>
@@ -14,4 +15,7 @@
     <xacro:property name="wheel_width" value="${20*mm2m}"/>
     <xacro:property name="caster_wheel_radius" value="${10*mm2m}"/>
+    <xacro:property name="lidar_radius" value="${50*mm2m}"/>
+    <xacro:property name="lidar_width" value="${20*mm2m}"/>
+    <xacro:property name="lidar_base" value="${30*mm2m}"/>
     <!-- ============= -->
     <!-- === WORLD === -->
@@ -93,3 +97,16 @@
         material_name="white"
     />
+    <!-- ============= -->
+    <!-- === LIDAR === -->
+    <!-- ============= -->
+    <xacro:lidar
+        name="lidar"
+        parent="base_link"
+        xyz="0 0 ${base_height/2+lidar_width/2+lidar_base}"
+        rpy="0 0 0"
+        radius="${lidar_radius}"
+        width="${lidar_width}"
+        m="0.1"
+        material_name="orange"
+    />
 </robot>

Commit message: feat: add LIDAR data transfer from Gazebo to rviz

File: twr_description/urdf/gz.xacro (robot description, xacro)
@@ -18,5 +18,5 @@
     <!-- === LIDAR === -->
     <gazebo reference="lidar_link">
-        <sensor name="lidar_link" type="gpu_lidar">
+        <sensor name="lidar" type="gpu_lidar">
             <pose> 0 0 0 0 0 0 </pose>
             <visualize>true</visualize>
@@ -31,10 +31,10 @@
                 </scan>
                 <range>
-                    <min>0.3</min>
-                    <max>10</max>
+                    <min>0.05</min>
+                    <max>5</max>
                 </range>
             </lidar>
             <topic>scan</topic>
-            <!-- <gz_frame_id>lidar_link</gz_frame_id> -->
+            <gz_frame_id>lidar_link</gz_frame_id>
         </sensor>
     </gazebo>

File: twr_description/urdf/twr.urdf.xacro (robot description, xacro)
@@ -15,7 +15,7 @@
     <xacro:property name="wheel_width" value="${20*mm2m}"/>
     <xacro:property name="caster_wheel_radius" value="${10*mm2m}"/>
-    <xacro:property name="lidar_radius" value="${50*mm2m}"/>
+    <xacro:property name="lidar_radius" value="${10*mm2m}"/>
     <xacro:property name="lidar_width" value="${20*mm2m}"/>
-    <xacro:property name="lidar_base" value="${30*mm2m}"/>
+    <xacro:property name="lidar_base" value="${60*mm2m}"/>
     <!-- ============= -->
     <!-- === WORLD === -->
