Commit message: style: update rviz config file, colors in urdf file

File: twr_description/urdf/twr.urdf.xacro (robot description, xacro)
@@ -23,5 +23,5 @@
         <parent link="odom"/>
         <child link="base_link" />
-        <origin xyz="0 0 ${wheel_radius+0.01}" rpy="0 0 0"/>
+        <origin xyz="0 0 ${wheel_radius+0.001}" rpy="0 0 0"/>
     </joint>
     <link name="base_link">
@@ -57,5 +57,5 @@
                 <cylinder radius="${wheel_radius}" length="${wheel_width}"/>
             </geometry>
-            <material name="white"/>
+            <material name="orange"/>
             <origin xyz="0 0 0" rpy="0 0 0"/>
         </visual>
@@ -66,5 +66,5 @@
             <origin xyz="0 0 0" rpy="0 0 0"/>
         </collision>
-        <xacro:cylinder_inertia m="1" r="${wheel_radius}" l="${wheel_width}">
+        <xacro:cylinder_inertia m="0.2" r="${wheel_radius}" l="${wheel_width}">
             <origin xyz="0 0 0" rpy="-${pi/2} 0 0"/>
         </xacro:cylinder_inertia>
@@ -81,5 +81,5 @@
                 <cylinder radius="${wheel_radius}" length="${wheel_width}"/>
             </geometry>
-            <material name="white"/>
+            <material name="orange"/>
             <origin xyz="0 0 0" rpy="0 0 0"/>
         </visual>
@@ -90,5 +90,5 @@
             <origin xyz="0 0 0" rpy="0 0 0"/>
         </collision>
-        <xacro:cylinder_inertia m="1" r="${wheel_radius}" l="${wheel_width}">
+        <xacro:cylinder_inertia m="0.2" r="${wheel_radius}" l="${wheel_width}">
             <origin xyz="0 0 0" rpy="${pi/2} 0 0"/>
         </xacro:cylinder_inertia>

Commit message: refactor(urdf): add xacro macro for wheel

File: twr_description/urdf/twr.urdf.xacro (robot description, xacro)
@@ -6,4 +6,5 @@
     <xacro:include filename="ros2_control.xacro"/>
     <xacro:include filename="gz.xacro"/>
+    <xacro:include filename="wheel.xacro"/>
     <xacro:property name="mm2m" value="0.001"/>
     <xacro:property name="base_length" value="${200*mm2m}"/>
@@ -46,52 +47,26 @@
     <!-- === WHEELS === -->
     <!-- ============== -->
-    <joint name="left_wheel_joint" type="continuous">
-        <parent link="base_link"/>
-        <child link="left_wheel_link" />
-        <origin xyz="0 ${base_width/2 + wheel_width/2 + 0.01} 0" rpy="-${pi/2} 0 0"/>
-        <axis xyz="0 0 1"/>
-    </joint>
-    <link name="left_wheel_link">
-        <visual>
-            <geometry>
-                <cylinder radius="${wheel_radius}" length="${wheel_width}"/>
-            </geometry>
-            <material name="orange"/>
-            <origin xyz="0 0 0" rpy="0 0 0"/>
-        </visual>
-        <collision>
-            <geometry>
-                <cylinder radius="${wheel_radius}" length="${wheel_width}"/>
-            </geometry>
-            <origin xyz="0 0 0" rpy="0 0 0"/>
-        </collision>
-        <xacro:cylinder_inertia m="0.2" r="${wheel_radius}" l="${wheel_width}">
-            <origin xyz="0 0 0" rpy="-${pi/2} 0 0"/>
-        </xacro:cylinder_inertia>
-    </link>
-    <joint name="right_wheel_joint" type="continuous">
-        <parent link="base_link"/>
-        <child link="right_wheel_link" />
-        <origin xyz="0 -${base_width/2 + wheel_width/2 + 0.01} 0" rpy="-${pi/2} 0 0"/>
-        <axis xyz="0 0 1"/>
-    </joint>
-    <link name="right_wheel_link">
-        <visual>
-            <geometry>
-                <cylinder radius="${wheel_radius}" length="${wheel_width}"/>
-            </geometry>
-            <material name="orange"/>
-            <origin xyz="0 0 0" rpy="0 0 0"/>
-        </visual>
-        <collision>
-            <geometry>
-                <cylinder radius="${wheel_radius}" length="${wheel_width}"/>
-            </geometry>
-            <origin xyz="0 0 0" rpy="0 0 0"/>
-        </collision>
-        <xacro:cylinder_inertia m="0.2" r="${wheel_radius}" l="${wheel_width}">
-            <origin xyz="0 0 0" rpy="${pi/2} 0 0"/>
-        </xacro:cylinder_inertia>
-    </link>
+    <xacro:wheel
+        name="left_wheel"
+        parent="base_link"
+        xyz="0 ${base_width/2 + wheel_width/2 + 0.01} 0"
+        rpy="-${pi/2} 0 0"
+        radius="${wheel_radius}"
+        width="${wheel_width}"
+        m="0.2"
+        xyz_axis="0 0 1"
+        material_name="orange"
+    />
+    <xacro:wheel
+        name="right_wheel"
+        parent="base_link"
+        xyz="0 -${base_width/2 + wheel_width/2 + 0.01} 0"
+        rpy="-${pi/2} 0 0"
+        radius="${wheel_radius}"
+        width="${wheel_width}"
+        m="0.2"
+        xyz_axis="0 0 1"
+        material_name="orange"
+    />
     <!-- ===================== -->
     <!-- === CASTER WHEELS === -->

Commit message: refactor(urdf): add type for xacro wheel macro, rename file

File: twr_description/urdf/twr.urdf.xacro (robot description, xacro)
@@ -49,4 +49,5 @@
     <xacro:wheel
         name="left_wheel"
+        type="standart"
         parent="base_link"
         xyz="0 ${base_width/2 + wheel_width/2 + 0.01} 0"
@@ -60,4 +61,5 @@
     <xacro:wheel
         name="right_wheel"
+        type="standart"
         parent="base_link"
         xyz="0 -${base_width/2 + wheel_width/2 + 0.01} 0"
@@ -69,54 +71,27 @@
         material_name="orange"
     />
-    <!-- ===================== -->
-    <!-- === CASTER WHEELS === -->
-    <!-- ===================== -->
-    <joint name="caster_front_wheel_joint" type="fixed">
-        <parent link="base_link"/>
-        <child link="caster_front_wheel_link"/>
-        <origin xyz="${base_length/2-caster_wheel_radius} 0 -${wheel_radius-caster_wheel_radius-1*mm2m}" rpy="0 0 0"/>
-        <axis xyz="1 1 1"/>
-    </joint>
-    <link name="caster_front_wheel_link">
-        <visual>
-            <geometry>
-                <sphere radius="${caster_wheel_radius}"/>
-            </geometry>
-            <material name="white"/>
-            <origin xyz="0 0 0" rpy="0 0 0"/>
-        </visual>
-        <collision>
-            <geometry>
-                <sphere radius="${caster_wheel_radius}"/>
-            </geometry>
-            <origin xyz="0 0 0" rpy="0 0 0"/>
-        </collision>
-        <xacro:sphere_inertia m="0.01" r="${caster_wheel_radius}">
-            <origin xyz="0 0 0" rpy="0 0 0"/>
-        </xacro:sphere_inertia>
-    </link>
-    <joint name="caster_back_wheel_joint" type="fixed">
-        <parent link="base_link"/>
-        <child link="caster_back_wheel_link"/>
-        <origin xyz="-${base_length/2-caster_wheel_radius} 0 -${wheel_radius-caster_wheel_radius-1*mm2m}" rpy="0 0 0"/>
-        <axis xyz="1 1 1"/>
-    </joint>
-    <link name="caster_back_wheel_link">
-        <visual>
-            <geometry>
-                <sphere radius="${caster_wheel_radius}"/>
-            </geometry>
-            <material name="white"/>
-            <origin xyz="0 0 0" rpy="0 0 0"/>
-        </visual>
-        <collision>
-            <geometry>
-                <sphere radius="${caster_wheel_radius}"/>
-            </geometry>
-            <origin xyz="0 0 0" rpy="0 0 0"/>
-        </collision>
-        <xacro:sphere_inertia m="0.01" r="${caster_wheel_radius}">
-            <origin xyz="0 0 0" rpy="0 0 0"/>
-        </xacro:sphere_inertia>
-    </link>
+    <xacro:wheel
+        name="caster_front_wheel"
+        type="caster"
+        parent="base_link"
+        xyz="${base_length/2-caster_wheel_radius} 0 -${wheel_radius-caster_wheel_radius-1*mm2m}"
+        rpy="0 0 0"
+        radius="${caster_wheel_radius}"
+        width="${caster_wheel_radius}"
+        m="0.01"
+        xyz_axis="0 0 0"
+        material_name="white"
+    />
+    <xacro:wheel
+        name="caster_back_wheel"
+        type="caster"
+        parent="base_link"
+        xyz="-${base_length/2-caster_wheel_radius} 0 -${wheel_radius-caster_wheel_radius-1*mm2m}"
+        rpy="0 0 0"
+        radius="${caster_wheel_radius}"
+        width="${caster_wheel_radius}"
+        m="0.01"
+        xyz_axis="0 0 0"
+        material_name="white"
+    />
 </robot>

Commit message: feat: prepare urdf file for slam algorithms - new base_footprint, odom and map coordinate frames

File: twr_description/urdf/twr.urdf.xacro (robot description, xacro)
@@ -18,13 +18,28 @@
     <xacro:property name="lidar_width" value="${20*mm2m}"/>
     <xacro:property name="lidar_base" value="${60*mm2m}"/>
-    <!-- ============= -->
-    <!-- === WORLD === -->
-    <!-- ============= -->
+    <!-- ============ -->
+    <!-- === MAP === -->
+    <!-- ============ -->
+    <link name="map"/>
+    <!-- ============ -->
+    <!-- === ODOM === -->
+    <!-- ============ -->
+    <joint name="odom_joint" type="fixed">
+        <parent link="map"/>
+        <child link="odom" />
+        <origin xyz="0 0 0" rpy="0 0 0"/>
+    </joint>
     <link name="odom"/>
     <!-- ============ -->
     <!-- === BASE === -->
     <!-- ============ -->
+    <joint name="base_footprint_joint" type="fixed">
+        <parent link="odom"/>
+        <child link="base_footprint" />
+        <origin xyz="0 0 0" rpy="0 0 0"/>
+    </joint>
+    <link name="base_footprint"/>
     <joint name="base_joint" type="fixed">
-        <parent link="odom"/>
+        <parent link="base_footprint"/>
         <child link="base_link" />
         <origin xyz="0 0 ${wheel_radius+0.001}" rpy="0 0 0"/>

Commit message: refactor(urdf): change links sequence map->odom->base_link->base_footprint

File: twr_description/urdf/twr.urdf.xacro (robot description, xacro)
@@ -34,12 +34,6 @@
     <!-- === BASE === -->
     <!-- ============ -->
-    <joint name="base_footprint_joint" type="fixed">
+    <joint name="base_joint" type="fixed">
         <parent link="odom"/>
-        <child link="base_footprint" />
-        <origin xyz="0 0 0" rpy="0 0 0"/>
-    </joint>
-    <link name="base_footprint"/>
-    <joint name="base_joint" type="fixed">
-        <parent link="base_footprint"/>
         <child link="base_link" />
         <origin xyz="0 0 ${wheel_radius+0.001}" rpy="0 0 0"/>
@@ -61,4 +55,11 @@
         <xacro:inertia shape="box" xyz="0 0 0" rpy="0 0 0" l="${base_length}" w="${base_width}" h="${base_height}" m="1"/>
     </link>
+    <!-- Base Footprint -->
+    <joint name="base_footprint_joint" type="fixed">
+        <parent link="base_link"/>
+        <child link="base_footprint" />
+        <origin xyz="0 0 -${wheel_radius+0.001}" rpy="0 0 0"/>
+    </joint>
+    <link name="base_footprint"/>
     <!-- ============== -->
     <!-- === WHEELS === -->

Commit message: fix(urdf): remove links not related to the robot model

File: twr_description/urdf/twr.urdf.xacro (robot description, xacro)
@@ -19,25 +19,14 @@
     <xacro:property name="lidar_base" value="${60*mm2m}"/>
     <!-- ============ -->
-    <!-- === MAP === -->
+    <!-- === BASE === -->
     <!-- ============ -->
-    <link name="map"/>
-    <!-- ============ -->
-    <!-- === ODOM === -->
-    <!-- ============ -->
-    <joint name="odom_joint" type="fixed">
-        <parent link="map"/>
-        <child link="odom" />
+    <link name="base_link"/>
+    <!-- Base Frame -->
+    <joint name="base_frame_joint" type="fixed">
+        <parent link="base_link"/>
+        <child link="base_frame_link" />
         <origin xyz="0 0 0" rpy="0 0 0"/>
     </joint>
-    <link name="odom"/>
-    <!-- ============ -->
-    <!-- === BASE === -->
-    <!-- ============ -->
-    <joint name="base_joint" type="fixed">
-        <parent link="odom"/>
-        <child link="base_link" />
-        <origin xyz="0 0 ${wheel_radius+0.001}" rpy="0 0 0"/>
-    </joint>
-    <link name="base_link">
+    <link name="base_frame_link">
         <visual>
             <geometry>

Commit message: refactor: update urdf file structure

File: twr_description/urdf/twr.urdf.xacro (robot description, xacro)
@@ -1,117 +1,17 @@
 <?xml version="1.0"?>
 <robot name="twr" xmlns:xacro="http://ros.org/wiki/xacro">
-    <!-- Include files -->
-    <xacro:include filename="_inertia.macro.xacro"/>
-    <xacro:include filename="_colors.xacro"/>
-    <xacro:include filename="ros2_control.xacro"/>
-    <xacro:include filename="gz.xacro"/>
-    <xacro:include filename="wheel.macro.xacro"/>
-    <xacro:include filename="twr_lidar.xacro"/>
-    <xacro:property name="mm2m" value="0.001"/>
-    <xacro:property name="base_length" value="${200*mm2m}"/>
-    <xacro:property name="base_width" value="${200*mm2m}"/>
-    <xacro:property name="base_height" value="${40*mm2m}"/>
-    <xacro:property name="wheel_radius" value="${50*mm2m}"/>
-    <xacro:property name="wheel_width" value="${20*mm2m}"/>
-    <xacro:property name="caster_wheel_radius" value="${10*mm2m}"/>
-    <xacro:property name="lidar_radius" value="${10*mm2m}"/>
-    <xacro:property name="lidar_width" value="${20*mm2m}"/>
-    <xacro:property name="lidar_base" value="${60*mm2m}"/>
-    <!-- ============ -->
-    <!-- === BASE === -->
-    <!-- ============ -->
-    <link name="base_link"/>
-    <!-- Base Frame -->
-    <joint name="base_frame_joint" type="fixed">
-        <parent link="base_link"/>
-        <child link="base_frame_link" />
-        <origin xyz="0 0 0" rpy="0 0 0"/>
-    </joint>
-    <link name="base_frame_link">
-        <visual>
-            <geometry>
-                <box size="${base_length} ${base_width} ${base_height}"/>
-            </geometry>
-            <material name="white"/>
-            <origin xyz="0 0 0" rpy="0 0 0"/>
-        </visual>
-        <collision>
-            <geometry>
-                <box size="${base_length} ${base_width} ${base_height}"/>
-            </geometry>
-            <origin xyz="0 0 0" rpy="0 0 0"/>
-        </collision>
-        <xacro:inertia shape="box" xyz="0 0 0" rpy="0 0 0" l="${base_length}" w="${base_width}" h="${base_height}" m="1"/>
-    </link>
-    <!-- Base Footprint -->
-    <joint name="base_footprint_joint" type="fixed">
-        <parent link="base_link"/>
-        <child link="base_footprint" />
-        <origin xyz="0 0 -${wheel_radius+0.001}" rpy="0 0 0"/>
-    </joint>
-    <link name="base_footprint"/>
-    <!-- ============== -->
-    <!-- === WHEELS === -->
-    <!-- ============== -->
-    <xacro:wheel
-        name="left_wheel"
-        type="standart"
-        parent="base_link"
-        xyz="0 ${base_width/2 + wheel_width/2 + 0.01} 0"
-        rpy="-${pi/2} 0 0"
-        radius="${wheel_radius}"
-        width="${wheel_width}"
-        m="0.2"
-        xyz_axis="0 0 1"
-        material_name="orange"
-    />
-    <xacro:wheel
-        name="right_wheel"
-        type="standart"
-        parent="base_link"
-        xyz="0 -${base_width/2 + wheel_width/2 + 0.01} 0"
-        rpy="-${pi/2} 0 0"
-        radius="${wheel_radius}"
-        width="${wheel_width}"
-        m="0.2"
-        xyz_axis="0 0 1"
-        material_name="orange"
-    />
-    <xacro:wheel
-        name="caster_front_wheel"
-        type="caster"
-        parent="base_link"
-        xyz="${base_length/2-caster_wheel_radius} 0 -${wheel_radius-caster_wheel_radius-1*mm2m}"
-        rpy="0 0 0"
-        radius="${caster_wheel_radius}"
-        width="${caster_wheel_radius}"
-        m="0.01"
-        xyz_axis="0 0 0"
-        material_name="white"
-    />
-    <xacro:wheel
-        name="caster_back_wheel"
-        type="caster"
-        parent="base_link"
-        xyz="-${base_length/2-caster_wheel_radius} 0 -${wheel_radius-caster_wheel_radius-1*mm2m}"
-        rpy="0 0 0"
-        radius="${caster_wheel_radius}"
-        width="${caster_wheel_radius}"
-        m="0.01"
-        xyz_axis="0 0 0"
-        material_name="white"
-    />
-    <!-- ============= -->
-    <!-- === LIDAR === -->
-    <!-- ============= -->
-    <xacro:lidar
-        name="lidar"
-        parent="base_link"
-        xyz="0 0 ${base_height/2+lidar_width/2+lidar_base}"
-        rpy="0 0 0"
-        radius="${lidar_radius}"
-        width="${lidar_width}"
-        m="0.1"
-        material_name="orange"
-    />
+  <xacro:include filename="$(find twr_description)/urdf/macros/inertia.macro.xacro"/>
+  <xacro:include filename="$(find twr_description)/urdf/macros/wheel.macro.xacro"/>
+  <xacro:include filename="$(find twr_description)/urdf/macros/lidar.macro.xacro"/>
+  <xacro:include filename="$(find twr_description)/urdf/packages/gz.xacro"/>
+  <xacro:include filename="$(find twr_description)/urdf/packages/ros2_control.xacro"/>
+  <xacro:include filename="$(find twr_description)/urdf/properties/colors.xacro"/>
+  <xacro:include filename="$(find twr_description)/urdf/properties/geometry.xacro"/>
+  <!-- === BASE === -->
+  <xacro:include filename="$(find twr_description)/urdf/parts/twr_base.xacro"/>
+  <!-- === WHEELS === -->
+  <xacro:include filename="$(find twr_description)/urdf/parts/twr_drive_wheels.xacro"/>
+  <xacro:include filename="$(find twr_description)/urdf/parts/twr_caster_wheels.xacro"/>
+  <!-- === SENSORS === -->
+  <xacro:include filename="$(find twr_description)/urdf/parts/sensors/twr_lidar.xacro"/>
 </robot>
