Commit message: feat: update parameters and design of robot

File: twr_description/urdf/macros/lidar.macro.xacro (robot description, xacro)
@@ -21,5 +21,12 @@
         <origin xyz="0 0 0" rpy="0 0 0"/>
       </collision>
-      <xacro:inertia shape="cylinder" xyz="0 0 0" rpy="0 0 0" r="${radius}" w="${width}" m="${m}"/>
+      <xacro:inertia
+        shape="cylinder"
+        xyz="0 0 0"
+        rpy="0 0 0"
+        r="${radius}"
+        w="${width}"
+        m="${m}"
+      />
     </link>
   </xacro:macro>

File: twr_description/urdf/macros/wheel.macro.xacro (robot description, xacro)
@@ -26,5 +26,12 @@
           <origin xyz="0 0 0" rpy="0 0 0"/>
         </collision>
-        <xacro:inertia shape="cylinder" xyz="0 0 0" rpy="0 0 0" r="${radius}" w="${width}" m="${m}"/>
+        <xacro:inertia
+          shape="cylinder"
+          xyz="0 0 0"
+          rpy="0 0 0"
+          r="${radius}"
+          w="${width}"
+          m="${m}"
+        />
       </link>
     </xacro:if>
@@ -41,5 +48,5 @@
         <visual>
           <geometry>
-            <sphere radius="${radius}"/>
+            <cylinder radius="${radius}" length="${width}"/>
           </geometry>
           <material name="${material_name}"/>
@@ -48,9 +55,20 @@
         <collision>
           <geometry>
-            <sphere radius="${radius}"/>
+            <cylinder radius="${radius}" length="${width}"/>
           </geometry>
           <origin xyz="0 0 0" rpy="0 0 0"/>
         </collision>
-        <xacro:inertia shape="sphere" xyz="0 0 0" rpy="0 0 0" r="${radius}" m="${m}"/>
+        <xacro:inertia
+          shape="cylinder"
+          xyz="0 0 0"
+          rpy="0 0 0"
+          r="${radius}"
+          w="${width}"
+          m="${m}"
+        />
+        <gazebo reference="${name}_link">
+          <mu1>0</mu1>
+          <mu2>0</mu2>
+        </gazebo>
       </link>
     </xacro:if>

File: twr_description/urdf/parts/sensors/twr_lidar.xacro (robot description, xacro)
@@ -4,10 +4,10 @@
     name="lidar"
     parent="base_link"
-    xyz="0 0 ${base_height/2+lidar_width/2+lidar_base}"
+    xyz="0 0 ${chassis_height + lidar_width/2 + 5*mm2m}"
     rpy="0 0 0"
     radius="${lidar_radius}"
     width="${lidar_width}"
     m="0.1"
-    material_name="orange"
+    material_name="black"
   />
 </robot>

File: twr_description/urdf/parts/twr_base.xacro (robot description, xacro)
@@ -3,24 +3,31 @@
   <link name="base_link"/>
   <!-- Base Frame -->
-  <joint name="base_frame_joint" type="fixed">
+  <joint name="chassis_joint" type="fixed">
     <parent link="base_link"/>
-    <child link="base_frame_link" />
+    <child link="chassis_link" />
     <origin xyz="0 0 0" rpy="0 0 0"/>
   </joint>
-  <link name="base_frame_link">
+  <link name="chassis_link">
     <visual>
       <geometry>
-        <box size="${base_length} ${base_width} ${base_height}"/>
+        <mesh filename="file://$(find twr_description)/mesh/twr_base.dae"/>
       </geometry>
-      <material name="white"/>
       <origin xyz="0 0 0" rpy="0 0 0"/>
     </visual>
     <collision>
       <geometry>
-        <box size="${base_length} ${base_width} ${base_height}"/>
+        <mesh filename="file://$(find twr_description)/mesh/twr_base.dae"/>
       </geometry>
       <origin xyz="0 0 0" rpy="0 0 0"/>
     </collision>
-    <xacro:inertia shape="box" xyz="0 0 0" rpy="0 0 0" l="${base_length}" w="${base_width}" h="${base_height}" m="1"/>
+    <xacro:inertia
+      shape="box"
+      xyz="0 0 ${chassis_height/2}"
+      rpy="0 0 0"
+      l="${chassis_length}"
+      w="${chassis_width}"
+      h="${chassis_height}"
+      m="1"
+    />
   </link>
   <!-- Base Footprint -->
@@ -28,5 +35,5 @@
     <parent link="base_link"/>
     <child link="base_footprint" />
-    <origin xyz="0 0 -${wheel_radius+0.001}" rpy="0 0 0"/>
+    <origin xyz="0 0 ${-drive_wheel_radius + drive_wheel_axis_offset}" rpy="0 0 0"/>
   </joint>
   <link name="base_footprint"/>

File: twr_description/urdf/parts/twr_caster_wheels.xacro (robot description, xacro)
@@ -2,26 +2,50 @@
 <robot xmlns:xacro="http://www.ros.org/wiki/xacro" >
   <xacro:wheel
-    name="caster_front_wheel"
+    name="caster_front_left_wheel"
     type="caster"
     parent="base_link"
-    xyz="${base_length/2-caster_wheel_radius} 0 -${wheel_radius-caster_wheel_radius-1*mm2m}"
-    rpy="0 0 0"
+    xyz="${chassis_length/3} ${chassis_width/3} ${-drive_wheel_radius + drive_wheel_axis_offset + caster_wheel_radius + 1*mm2m}"
+    rpy="${pi/2} 0 0"
     radius="${caster_wheel_radius}"
-    width="${caster_wheel_radius}"
+    width="${caster_wheel_width}"
     m="0.01"
     xyz_axis="0 0 0"
-    material_name="white"
+    material_name="orange"
   />
   <xacro:wheel
-    name="caster_back_wheel"
+    name="caster_front_right_wheel"
     type="caster"
     parent="base_link"
-    xyz="-${base_length/2-caster_wheel_radius} 0 -${wheel_radius-caster_wheel_radius-1*mm2m}"
-    rpy="0 0 0"
+    xyz="${chassis_length/3} ${-chassis_width/3} ${-drive_wheel_radius + drive_wheel_axis_offset + caster_wheel_radius + 1*mm2m}"
+    rpy="${pi/2} 0 0"
     radius="${caster_wheel_radius}"
-    width="${caster_wheel_radius}"
+    width="${caster_wheel_width}"
     m="0.01"
     xyz_axis="0 0 0"
-    material_name="white"
+    material_name="orange"
+  />
+  <xacro:wheel
+    name="caster_back_left_wheel"
+    type="caster"
+    parent="base_link"
+    xyz="${-chassis_length/3} ${chassis_width/3} ${-drive_wheel_radius + drive_wheel_axis_offset + caster_wheel_radius + 1*mm2m}"
+    rpy="${pi/2} 0 0"
+    radius="${caster_wheel_radius}"
+    width="${caster_wheel_width}"
+    m="0.01"
+    xyz_axis="0 0 0"
+    material_name="orange"
+  />
+  <xacro:wheel
+    name="caster_back_right_wheel"
+    type="caster"
+    parent="base_link"
+    xyz="${-chassis_length/3} ${-chassis_width/3} ${-drive_wheel_radius + drive_wheel_axis_offset + caster_wheel_radius + 1*mm2m}"
+    rpy="${pi/2} 0 0"
+    radius="${caster_wheel_radius}"
+    width="${caster_wheel_width}"
+    m="0.01"
+    xyz_axis="0 0 0"
+    material_name="orange"
   />
 </robot>

File: twr_description/urdf/parts/twr_drive_wheels.xacro (robot description, xacro)
@@ -5,8 +5,8 @@
     type="drive"
     parent="base_link"
-    xyz="0 ${base_width/2 + wheel_width/2 + 0.01} 0"
-    rpy="-${pi/2} 0 0"
-    radius="${wheel_radius}"
-    width="${wheel_width}"
+    xyz="0 ${track_width/2} ${drive_wheel_axis_offset}"
+    rpy="${-pi/2} 0 0"
+    radius="${drive_wheel_radius}"
+    width="${drive_wheel_width}"
     m="0.2"
     xyz_axis="0 0 1"
@@ -17,8 +17,8 @@
     type="drive"
     parent="base_link"
-    xyz="0 -${base_width/2 + wheel_width/2 + 0.01} 0"
-    rpy="-${pi/2} 0 0"
-    radius="${wheel_radius}"
-    width="${wheel_width}"
+    xyz="0 ${-track_width/2} ${drive_wheel_axis_offset}"
+    rpy="${-pi/2} 0 0"
+    radius="${drive_wheel_radius}"
+    width="${drive_wheel_width}"
     m="0.2"
     xyz_axis="0 0 1"

File: twr_description/urdf/properties/geometry.xacro (robot description, xacro)
@@ -2,12 +2,14 @@
 <robot xmlns:xacro="http://www.ros.org/wiki/xacro" >
   <xacro:property name="mm2m" value="0.001"/>
-  <xacro:property name="base_length" value="${200*mm2m}"/>
-  <xacro:property name="base_width" value="${200*mm2m}"/>
-  <xacro:property name="base_height" value="${40*mm2m}"/>
-  <xacro:property name="wheel_radius" value="${50*mm2m}"/>
-  <xacro:property name="wheel_width" value="${20*mm2m}"/>
-  <xacro:property name="caster_wheel_radius" value="${10*mm2m}"/>
-  <xacro:property name="lidar_radius" value="${10*mm2m}"/>
+  <xacro:property name="chassis_length" value="${700*mm2m}"/>
+  <xacro:property name="chassis_width" value="${550*mm2m}"/>
+  <xacro:property name="chassis_height" value="${175*mm2m}"/>
+  <xacro:property name="drive_wheel_radius" value="${80*mm2m}"/>
+  <xacro:property name="drive_wheel_width" value="${40*mm2m}"/>
+  <xacro:property name="drive_wheel_axis_offset" value="${50*mm2m}"/>
+  <xacro:property name="track_width" value="${chassis_width - drive_wheel_width}"/>
+  <xacro:property name="caster_wheel_radius" value="${20*mm2m}"/>
+  <xacro:property name="caster_wheel_width" value="${15*mm2m}"/>
+  <xacro:property name="lidar_radius" value="${30*mm2m}"/>
   <xacro:property name="lidar_width" value="${20*mm2m}"/>
-  <xacro:property name="lidar_base" value="${60*mm2m}"/>
 </robot>
