Commit message: fix: raise robot base for correct display in rviz

File: twr_description/urdf/parts/sensors/twr_lidar.xacro (robot description, xacro)
@@ -3,5 +3,5 @@
   <xacro:lidar
     name="lidar"
-    parent="base_link"
+    parent="chassis_link"
     xyz="0 0 ${chassis_height + lidar_width/2 + 5*mm2m}"
     rpy="0 0 0"

File: twr_description/urdf/parts/twr_base.xacro (robot description, xacro)
@@ -1,10 +1,11 @@
 <?xml version="1.0"?>
 <robot xmlns:xacro="http://ros.org/wiki/xacro">
+  <!-- Base Frame -->
   <link name="base_link"/>
-  <!-- Base Frame -->
+  <!-- Chassis Frame -->
   <joint name="chassis_joint" type="fixed">
     <parent link="base_link"/>
     <child link="chassis_link" />
-    <origin xyz="0 0 0" rpy="0 0 0"/>
+    <origin xyz="0 0 ${drive_wheel_radius - drive_wheel_axis_offset}" rpy="0 0 0"/>
   </joint>
   <link name="chassis_link">
@@ -35,5 +36,5 @@
     <parent link="base_link"/>
     <child link="base_footprint" />
-    <origin xyz="0 0 ${-drive_wheel_radius + drive_wheel_axis_offset}" rpy="0 0 0"/>
+    <origin xyz="0 0 0" rpy="0 0 0"/>
   </joint>
   <link name="base_footprint"/>

File: twr_description/urdf/parts/twr_caster_wheels.xacro (robot description, xacro)
@@ -4,5 +4,5 @@
     name="caster_front_left_wheel"
     type="caster"
-    parent="base_link"
+    parent="chassis_link"
     xyz="${chassis_length/3} ${chassis_width/3} ${-drive_wheel_radius + drive_wheel_axis_offset + caster_wheel_radius + 1*mm2m}"
     rpy="${pi/2} 0 0"
@@ -16,5 +16,5 @@
     name="caster_front_right_wheel"
     type="caster"
-    parent="base_link"
+    parent="chassis_link"
     xyz="${chassis_length/3} ${-chassis_width/3} ${-drive_wheel_radius + drive_wheel_axis_offset + caster_wheel_radius + 1*mm2m}"
     rpy="${pi/2} 0 0"
@@ -28,5 +28,5 @@
     name="caster_back_left_wheel"
     type="caster"
-    parent="base_link"
+    parent="chassis_link"
     xyz="${-chassis_length/3} ${chassis_width/3} ${-drive_wheel_radius + drive_wheel_axis_offset + caster_wheel_radius + 1*mm2m}"
     rpy="${pi/2} 0 0"
@@ -40,5 +40,5 @@
     name="caster_back_right_wheel"
     type="caster"
-    parent="base_link"
+    parent="chassis_link"
     xyz="${-chassis_length/3} ${-chassis_width/3} ${-drive_wheel_radius + drive_wheel_axis_offset + caster_wheel_radius + 1*mm2m}"
     rpy="${pi/2} 0 0"

File: twr_description/urdf/parts/twr_drive_wheels.xacro (robot description, xacro)
@@ -4,5 +4,5 @@
     name="left_wheel"
     type="drive"
-    parent="base_link"
+    parent="chassis_link"
     xyz="0 ${track_width/2} ${drive_wheel_axis_offset}"
     rpy="${-pi/2} 0 0"
@@ -16,5 +16,5 @@
     name="right_wheel"
     type="drive"
-    parent="base_link"
+    parent="chassis_link"
     xyz="0 ${-track_width/2} ${drive_wheel_axis_offset}"
     rpy="${-pi/2} 0 0"
