Commit message: fix: change drive wheel width

File: twr_description/urdf/properties/geometry.xacro (robot description, xacro)
@@ -6,5 +6,5 @@
   <xacro:property name="chassis_height" value="${175*mm2m}"/>
   <xacro:property name="drive_wheel_radius" value="${80*mm2m}"/>
-  <xacro:property name="drive_wheel_width" value="${40*mm2m}"/>
+  <xacro:property name="drive_wheel_width" value="${20*mm2m}"/>
   <xacro:property name="drive_wheel_axis_offset" value="${50*mm2m}"/>
   <xacro:property name="track_width" value="${chassis_width - drive_wheel_width}"/>
