Commit message: feat: add gazebo imu sensor

File: twr_description/urdf/packages/gz.xacro (robot description, xacro)
@@ -27,4 +27,13 @@
     </sensor>
   </gazebo>
+  <!-- === IMU === -->
+  <gazebo reference="imu_link">
+    <sensor name="imu" type="imu">
+      <always_on>true</always_on>
+      <update_rate>10</update_rate>
+      <visualize>true</visualize>
+      <topic>imu</topic>
+    </sensor>
+  </gazebo>
   <!-- =============== -->
   <!-- === Plugins === -->
@@ -47,4 +56,7 @@
       <dimensions>3</dimensions>
     </plugin>
+    <plugin
+      filename="gz-sim-imu-system" name="gz::sim::systems::Imu">
+    </plugin>
   </gazebo>
 </robot>

File: twr_description/urdf/properties/geometry.xacro (robot description, xacro)
@@ -13,3 +13,6 @@
   <xacro:property name="lidar_radius" value="${30*mm2m}"/>
   <xacro:property name="lidar_width" value="${20*mm2m}"/>
+  <xacro:property name="imu_length" value="${10*mm2m}"/>
+  <xacro:property name="imu_width" value="${10*mm2m}"/>
+  <xacro:property name="imu_height" value="${10*mm2m}"/>
 </robot>

File: twr_description/urdf/twr.urdf.xacro (robot description, xacro)
@@ -15,3 +15,4 @@
   <!-- === SENSORS === -->
   <xacro:include filename="$(find twr_description)/urdf/parts/sensors/twr_lidar.xacro"/>
+  <xacro:include filename="$(find twr_description)/urdf/parts/sensors/twr_imu.xacro"/>
 </robot>
