Commit message: feat(mesh): update mesh file format to .OBJ for both URDF and MJCF

File: twr_description/urdf/parts/twr_base.xacro (robot description, xacro)
@@ -12,5 +12,5 @@
     <visual>
       <geometry>
-        <mesh filename="file://$(find twr_description)/mesh/twr_base.dae"/>
+        <mesh filename="file://$(find twr_description)/mesh/twr_base.obj" scale="0.001 0.001 0.001"/>
       </geometry>
       <origin xyz="0 0 0" rpy="0 0 0"/>
@@ -18,5 +18,5 @@
     <collision>
       <geometry>
-        <mesh filename="file://$(find twr_description)/mesh/twr_base.dae"/>
+        <mesh filename="file://$(find twr_description)/mesh/twr_base.obj" scale="0.001 0.001 0.001"/>
       </geometry>
       <origin xyz="0 0 0" rpy="0 0 0"/>
